Commit message: changed the visibility to public

File: softmatics_description/urdf/softmatics.xacro (robot description, xacro)
@@ -11,5 +11,5 @@
         <origin xyz="0 0 0" rpy="0 0 0" />
         <geometry>
-          <mesh filename="package://softmatics_visualization/meshes/visual/base.stl" />
+          <mesh filename="package://softmatics_description/meshes/visual/base.stl" />
         </geometry>
         <material name="">
@@ -20,5 +20,5 @@
         <origin xyz="0 0 0" rpy="0 0 0" />
         <geometry>
-          <mesh filename="package://softmatics_visualization/meshes/collision/base.stl" />
+          <mesh filename="package://softmatics_description/meshes/collision/base.stl" />
         </geometry>
       </collision>

File: softmatics_description/urdf/softmatics_model.xacro (robot description, xacro)
@@ -1,5 +1,5 @@
 <?xml version="1.0"?>
 <robot name="softmatics_model" xmlns:xacro="http://ros.org/wiki/xacro">
-  <xacro:include filename="$(find softmatics_visualization)/urdf/softmatics_model_macro.xacro" />
+  <xacro:include filename="$(find softmatics_description)/urdf/softmatics_model_macro.xacro" />
   <xacro:softmatics prefix=""/>
 </robot>

File: softmatics_description/urdf/softmatics_model_macro.xacro (robot description, xacro)
@@ -1,5 +1,5 @@
 <?xml version="1.0"?>
 <robot xmlns:xacro="http://ros.org/wiki/xacro">
-  <xacro:include filename="$(find softmatics_visualization)/urdf/softmatics_transmission.xacro" />
+  <xacro:include filename="$(find softmatics_description)/urdf/softmatics_transmission.xacro" />
   <xacro:macro name="knuckle" params="prefix fingerprefix">
     <link name="${prefix}${fingerprefix}_knuckle">
@@ -12,5 +12,5 @@
         <origin xyz="0 0 0" rpy="0 0 0" />
         <geometry>
-          <mesh filename="package://softmatics_visualization/meshes/visual/finger.stl" />
+          <mesh filename="package://softmatics_description/meshes/visual/finger.stl" />
         </geometry>
         <material name="">
@@ -21,10 +21,10 @@
         <origin xyz="0 0 0" rpy="0 0 0" />
         <geometry>
-          <mesh filename="package://softmatics_visualization/meshes/collision/finger.stl" />
+          <mesh filename="package://softmatics_description/meshes/collision/finger.stl" />
         </geometry>
       </collision>
     </link>
   </xacro:macro>
-  <xacro:include filename="$(find softmatics_visualization)/urdf/softmatics.xacro" />
+  <xacro:include filename="$(find softmatics_description)/urdf/softmatics.xacro" />
   <xacro:macro name="knuckle_joint" params="prefix">
     <joint name="${prefix}knuckle_joint" type="revolute">

File: softmatics_description/urdf/softmatics_transmission.xacro (robot description, xacro)
@@ -5,7 +5,8 @@
       <type>transmission_interface/SimpleTransmission</type>
       <joint name="${prefix}knuckle_joint">
-        <hardwareInterface>PositionJointInterface</hardwareInterface>
+        <hardwareInterface>hardware_interface/EffortJointInterface</hardwareInterface>
       </joint>
       <actuator name="${prefix}knuckle_joint_motor">
+        <hardwareInterface>hardware_interface/EffortJointInterface</hardwareInterface>
         <mechanicalReduction>1</mechanicalReduction>
       </actuator>

Commit message: add gazebo

File: softmatics_description/urdf/softmatics.xacro (robot description, xacro)
@@ -11,5 +11,5 @@
         <origin xyz="0 0 0" rpy="0 0 0" />
         <geometry>
-          <mesh filename="package://softmatics_description/meshes/visual/base.stl" />
+          <mesh filename="package://softmatics_description/meshes/visual/root.stl" />
         </geometry>
         <material name="">
@@ -20,8 +20,53 @@
         <origin xyz="0 0 0" rpy="0 0 0" />
         <geometry>
-          <mesh filename="package://softmatics_description/meshes/collision/base.stl" />
+          <mesh filename="package://softmatics_description/meshes/collision/root.stl" />
         </geometry>
       </collision>
     </link>
+    <link name="${prefix}palm_link">
+      <inertial>
+        <origin xyz="0.0 0.0 0.0" rpy="0 0 0" />
+        <mass value="0.7" />
+        <inertia ixx="1.0E-03" ixy="1.0E-06" ixz="1.0E-06" iyy="1.0E-03" iyz="1.0E-06" izz="1.0E-03" />
+      </inertial>
+      <visual>
+        <origin xyz="0 0 0" rpy="0 0 0" />
+        <geometry>
+          <mesh filename="package://softmatics_description/meshes/visual/palm.stl" />
+        </geometry>
+        <material name="">
+          <color rgba="0.0 0.2 0.7 0.8" />
+        </material>
+      </visual>
+      <collision>
+        <origin xyz="0 0 0" rpy="0 0 0" />
+        <geometry>
+          <mesh filename="package://softmatics_description/meshes/collision/palm.stl" />
+        </geometry>
+      </collision>
+    </link>
+    <link name="world"/>
+    <joint name="joint0" type="fixed">
+      <parent link="world"/>
+      <child link="${prefix}softmatics_base_link"/>
+      <origin xyz= "0. 0. 0." rpy="0. 0. 0." />
+    </joint>
+    <joint name="${prefix}palm_joint" type="fixed">
+      <parent link="${prefix}softmatics_base_link"/>
+      <child link="${prefix}palm_link"/>
+      <origin xyz= "0. 0. 0." rpy="0. 0. 0." />
+    </joint>
+    <gazebo reference="${prefix}softmatics_base_link">
+      <mu1>1.0</mu1>
+      <mu2>1.0</mu2>
+      <selfCollide>false</selfCollide>
+      <material>Gazebo/White</material>
+    </gazebo>
+    <gazebo reference="${prefix}palm_link">
+      <mu1>1.0</mu1>
+      <mu2>1.0</mu2>
+      <selfCollide>false</selfCollide>
+      <material>Gazebo/SkyBlue</material>
+    </gazebo>
   </xacro:macro>
   <xacro:macro name="finger_links" params="prefix fingerprefix">

File: softmatics_description/urdf/softmatics_model_macro.xacro (robot description, xacro)
@@ -2,4 +2,5 @@
 <robot xmlns:xacro="http://ros.org/wiki/xacro">
   <xacro:include filename="$(find softmatics_description)/urdf/softmatics_transmission.xacro" />
+  <xacro:include filename="$(find softmatics_description)/urdf/softmatics_gazebo.xacro" />
   <xacro:macro name="knuckle" params="prefix fingerprefix">
     <link name="${prefix}${fingerprefix}_knuckle">
@@ -15,5 +16,5 @@
         </geometry>
         <material name="">
-          <color rgba="0.8 0.8 0.8 1" />
+          <color rgba="0.0 0.2 0.7 0.8" />
         </material>
       </visual>
@@ -25,4 +26,13 @@
       </collision>
     </link>
+    <gazebo reference="${prefix}${fingerprefix}_knuckle">
+      <kp>1000000.0</kp>
+      <kd>1.0</kd>
+      <mu1>1.0</mu1>
+      <mu2>1.0</mu2>
+      <minDepth>0.001</minDepth>
+      <selfCollide>false</selfCollide>
+      <material>Gazebo/SkyBlue</material>
+    </gazebo>
   </xacro:macro>
   <xacro:include filename="$(find softmatics_description)/urdf/softmatics.xacro" />
@@ -33,5 +43,5 @@
       <child link="${prefix}first_knuckle" />
       <axis xyz="-1 0 0" />
-      <limit lower="0.0" upper="0.872664" velocity="2.0" effort="1000" />
+      <limit lower="0.0" upper="0.872664" velocity="100.0" effort="1000" />
     </joint>
   </xacro:macro>
@@ -42,6 +52,6 @@
       <child link="${prefix}second_knuckle" />
       <axis xyz="-1 0 0" />
-      <limit lower="0.0" upper="0.872664" velocity="2.0" effort="1000" />
-    <mimic joint="${prefix}knuckle_joint" multiplier="1" offset="0" />
+      <limit lower="0.0" upper="0.872664" velocity="100.0" effort="1000" />
+      <mimic joint="${prefix}knuckle_joint" multiplier="1" offset="0" />
     </joint>
   </xacro:macro>
@@ -52,6 +62,6 @@
       <child link="${prefix}third_knuckle" />
       <axis xyz="-1 0 0" />
-      <limit lower="0.0" upper="0.872664" velocity="2.0" effort="1000" />
-    <mimic joint="${prefix}knuckle_joint" multiplier="1" offset="0" />
+      <limit lower="0.0" upper="0.872664" velocity="100.0" effort="1000" />
+      <mimic joint="${prefix}knuckle_joint" multiplier="1" offset="0" />
     </joint>
   </xacro:macro>
@@ -62,6 +72,6 @@
       <child link="${prefix}fourth_knuckle" />
       <axis xyz="-1 0 0" />
-      <limit lower="0.0" upper="0.872664" velocity="2.0" effort="1000" />
-    <mimic joint="${prefix}knuckle_joint" multiplier="1" offset="0" />
+      <limit lower="0.0" upper="0.872664" velocity="100.0" effort="1000" />
+      <mimic joint="${prefix}knuckle_joint" multiplier="1" offset="0" />
     </joint>
   </xacro:macro>
@@ -72,6 +82,6 @@
       <child link="${prefix}fifth_knuckle" />
       <axis xyz="-1 0 0" />
-      <limit lower="0.0" upper="0.872664" velocity="2.0" effort="1000" />
-    <mimic joint="${prefix}knuckle_joint" multiplier="1" offset="0" />
+      <limit lower="0.0" upper="0.872664" velocity="100.0" effort="1000" />
+      <mimic joint="${prefix}knuckle_joint" multiplier="1" offset="0" />
     </joint>
   </xacro:macro>
@@ -89,4 +99,5 @@
     <xacro:fifth_knuckle_joint prefix="${prefix}"/>
     <xacro:softmatics_transmission prefix="${prefix}"/>
+    <xacro:softmatics_gazebo prefix="${prefix}"/>
   </xacro:macro>
 </robot>
